Commit message: Camera angle fixed in gazebo

File: urdf/uma_grover.urdf (robot description, URDF)
Before this commit: robot uma_grover, 8 links, 7 joints
Joints:
- joint camera_joint: origin xyz=0.31 0.02652 0.18549 rpy=1.604 0 0 -> xyz=0.31 0.02050 0.18549 rpy=6.28319 0 4.71239

Commit message: Lidar and size of wheels fixed

File: urdf/uma_grover.urdf (robot description, URDF)
Before this commit: robot uma_grover, 8 links, 7 joints
Joints:
- joint lidar_joint: origin xyz=0.31 -0.03 0.02 rpy=1.5708 0 0.67324 -> xyz=0.31 -0.03 0.045 rpy=0 0 0; type continuous -> fixed

Commit message: Angular and linear velocity fixed

File: urdf/uma_grover.urdf (robot description, URDF)
Before this commit: robot uma_grover, 8 links, 7 joints
Joints:
- joint wbl_joint: axis 0 0 1 -> 0 0 -1
- joint wfl_joint: axis 0 0 1 -> 0 0 -1

Commit message: Fixed links and odom

File: urdf/uma_grover.urdf (robot description, URDF)
Before this commit: robot uma_grover, 8 links, 7 joints
Links:
- added link chassis_link, mass 13.426; collision mesh filename=package://uma_grover/meshes/base_link.STL; visual mesh filename=package://uma_grover/meshes/base_link.STL
- link base_link: mass 13.426 -> None; geometry 
Joints:
- added joint dummy joint: type fixed, parent base_link, child chassis_link, origin xyz=0 0 0 rpy=0 0 0
- joint camera_joint: parent base_link -> chassis_link
- joint lidar_joint: parent base_link -> chassis_link
- joint rtk_joint: parent base_link -> chassis_link
- joint wbl_joint: parent base_link -> chassis_link
- joint wbr_joint: parent base_link -> chassis_link
- joint wfl_joint: parent base_link -> chassis_link
- joint wfr_joint: parent base_link -> chassis_link

Commit message: Lidar fixed to 180 degrees

File: urdf/uma_grover.urdf (robot description, URDF)
Before this commit: robot uma_grover, 9 links, 8 joints
Joints:
- joint lidar_joint: origin xyz=0.31 -0.03 0.045 rpy=0 0 0 -> xyz=0.31 -0.03 0.045 rpy=0 0 4.71239

Commit message: Links base and rtk fixed

File: urdf/uma_grover.urdf (robot description, URDF)
Before this commit: robot uma_grover, 9 links, 8 joints
Joints:
- joint dummy joint: origin xyz=0 0 0 rpy=0 0 0 -> xyz=0.31 -0.31 0.1 rpy=0 0 1.5708
- joint rtk_joint: origin xyz=0.1025 0.088 0.47318 rpy=-1.5708 0 -1.5708 -> xyz=0.1025 0.088 0.47318 rpy=0 0 -1.5708
